File: bucker.sch (KiCad schematic (older format))
At the start: 29 parts, among them SW1 SW_SPDT, SW2 SW_DIP_x4, U1 TPS54231

Commit message: Added current sense amp and connector.
Parts:
- added C9: 0.1uF, Capacitors_SMD:C_0805_HandSoldering, symbol C_Small
- added J1: CONN_02X03, Pin_Headers:Pin_Header_Straight_2x03_Pitch2.54mm, symbol CONN_02X03
- added U2: LMP8640, TO_SOT_Packages_SMD:SOT-23-6_Handsoldering, symbol LMP8640
- C3: MFG Taiyo Yuden -> Murata; MFG PN (none) -> GRM216R71H103KA01D
- C4: MFG (none) -> Yageo; MFG PN (none) -> CC0805JRNPO9BN102; Package ID (none) -> 0805; Source (none) -> 311-1122-1-ND
- C5: MFG (none) -> Yageo
- C6: MFG (none) -> Yageo; MFG PN (none) -> CC0805JRNPO9BN470; Package ID (none) -> 0805; Source (none) -> 311-1107-1-ND
- D2: MFG (none) -> Lite-On
- L1: Description (none) -> 22uH, 2.2A 56mOhm; MFG (none) -> Bourns; MFG PN (none) -> SRU1038-220Y; Source (none) -> SRU1038-220YCT-ND
- R1, R3, R5: MFG (none) -> Yageo; MFG PN (none) -> RC0805FR-0710KL; Package ID (none) -> 0805
- R2: MFG (none) -> Yageo; MFG PN (none) -> RC0805FR-073K24L; Package ID (none) -> 0805; Source (none) -> 311-3.24KCRCT-ND
- R4: MFG (none) -> Yageo; MFG PN (none) -> RC0805FR-071K91L; Package ID (none) -> 0805; Source (none) -> 311-1.91KCRCT-ND
- R6: value 2k -> 2.2k; MFG (none) -> Yageo; MFG PN (none) -> RC0805FR-072K2L; Package ID (none) -> 0805; Source (none) -> 311-2.2KARCT-ND
- R7: MFG (none) -> Yageo; MFG PN (none) -> RC0805FR-0733KL; Package ID (none) -> 0805; Source (none) -> 311-33.0KCRCT-ND
- R8: MFG (none) -> Yageo; MFG PN (none) -> PE2512FKE070R1L; Package ID (none) -> 2512; Source (none) -> YAG2159CT-ND
- RV1: value POT -> 10k; MFG (none) -> Panasonic; MFG PN (none) -> EVM-3YSX50B14; Notes (none) -> EOL; Source (none) -> P3Y103CT-ND
Connections:
- net GND: now also J1.6 (P6)
- net VCC: now also J1.4 (P4)
- net VOUT: now also U2.3 (+IN)
- net at R8.1, TB2.1 (P1): now also U2.4 (-IN)
- new net: J1.1 (P1), U2.1 (Vout)
- new net INSTR_GND: C9.1, J1.5 (P5), U2.2 (V-)
- new net INSTR_VCC: C9.2, J1.3 (P3), U2.6 (V+)

Commit message: Aligned mounting holes and terminal blocks.
Parts:
- H1, H2: value M3 screw -> PLATED_HOLE; footprint Mounting_Holes:MountingHole_3.2mm_M3_Pad_Via -> Mounting_Holes:MountingHole_3.2mm_M3_Pad
Connections:
- net GND: now also H1.~, H2.~
Changed lines of the file:
@@
 Text Label 7200 1750 0    50   ~ 0
 VOUT
-$Comp
-L PLATED_HOLE H1
-U 1 1 58227CC3
-P 1450 6650
-F 0 "H1" H 1300 6650 50  0000 C CNN
-F 1 "M3 screw" H 1500 6550 50  0000 C CNN
-F 2 "Mounting_Holes:MountingHole_3.2mm_M3_Pad_Via" H 1450 6650 50  0001 C CNN
-F 3 "" H 1450 6650 50  0001 C CNN
-	1    1450 6650
-	1    0    0    -1
-$EndComp
-$Comp
-L PLATED_HOLE H2
-U 1 1 58227EDC
-P 2000 6650
-F 0 "H2" H 1850 6650 50  0000 C CNN
-F 1 "M3 screw" H 2050 6550 50  0000 C CNN
-F 2 "Mounting_Holes:MountingHole_3.2mm_M3_Pad_Via" H 2000 6650 50  0001 C CNN
-F 3 "" H 2000 6650 50  0001 C CNN
-	1    2000 6650
-	1    0    0    -1
-$EndComp
 Wire Wire Line
 	8750 1750 8750 1800
@@
 Wire Wire Line
 	10100 2750 10100 2850
+$Comp
+L GND #PWR017
+U 1 1 58B5B250
+P 1900 6900
+F 0 "#PWR017" H 1900 6650 50  0001 C CNN
+F 1 "GND" H 1900 6750 50  0000 C CNN
+F 2 "" H 1900 6900 50  0000 C CNN
+F 3 "" H 1900 6900 50  0000 C CNN
+	1    1900 6900
+	1    0    0    -1
+$EndComp
+Wire Wire Line
+	1450 6650 1450 6850
+Wire Wire Line
+	1450 6850 2000 6850
+Wire Wire Line
+	2000 6850 2000 6650
+Wire Wire Line
+	1900 6900 1900 6850
+Connection ~ 1900 6850
+$Comp
+L PLATED_HOLE H1
+U 1 1 58B5DAA7
+P 1450 6650
+F 0 "H1" H 1578 6815 50  0000 L CNN
+F 1 "PLATED_HOLE" H 1578 6724 50  0000 L CNN
+F 2 "Mounting_Holes:MountingHole_3.2mm_M3_Pad" H 500 150 50  0001 C CNN
+F 3 "" H 500 150 50  0001 C CNN
+	1    1450 6650
+	1    0    0    -1
+$EndComp
+$Comp
+L PLATED_HOLE H2
+U 1 1 58B5DB73
+P 2000 6650
+F 0 "H2" H 2128 6815 50  0000 L CNN
+F 1 "PLATED_HOLE" H 2128 6724 50  0000 L CNN
+F 2 "Mounting_Holes:MountingHole_3.2mm_M3_Pad" H 1050 150 50  0001 C CNN
+F 3 "" H 1050 150 50  0001 C CNN
+	1    2000 6650
+	1    0    0    -1
+$EndComp
 $EndSCHEMATC
